Commit message: checkpoint: sync current AMR simulation state

File: src/amr_description/urdf/amr.urdf.xacro (robot description, xacro)
@@ -36,4 +36,23 @@
   <xacro:property name="cad_body_rgba" value="0.752941176470588 0.752941176470588 0.752941176470588 1"/>
   <xacro:property name="cad_bluegray_rgba" value="0.792156862745098 0.819607843137255 0.933333333333333 1"/>
+  <!--
+    Gazebo Harmonic gpu_lidar uses the SDF visibility-mask / visual-flags
+    contract.  Bit 0 is reserved for geometry belonging to this robot; the
+    sensor mask accepts all other visibility bits.
+  -->
+  <xacro:property name="lidar_self_visibility_flag" value="1"/>
+  <xacro:property name="lidar_visibility_mask" value="4294967294"/>
+  <!--
+    The nested visual extension is applied to every visual on the referenced
+    link by the URDF-to-SDF converter.  Keep source visual elements unnamed so
+    the converter can merge this extension reliably across fixed-joint lumps.
+  -->
+  <xacro:macro name="exclude_lidar_self_visuals" params="link">
+    <gazebo reference="${link}">
+      <visual>
+        <visibility_flags>${lidar_self_visibility_flag}</visibility_flags>
+      </visual>
+    </gazebo>
+  </xacro:macro>
   <xacro:macro name="cad_material" params="name rgba">
     <material name="${name}">
@@ -61,5 +80,5 @@
   <xacro:macro name="drive_wheel" params="name y rpy axis_z">
     <link name="${name}">
-      <visual name="cad_visual">
+      <visual>
         <origin xyz="0 0 0" rpy="0 0 0"/>
         <geometry><mesh filename="package://amr_description/meshes/${name}_link.STL"/></geometry>
@@ -79,9 +98,10 @@
       <dynamics damping="0.7" friction="0.7"/>
     </joint>
+    <xacro:exclude_lidar_self_visuals link="${name}"/>
   </xacro:macro>
   <xacro:macro name="passive_caster" params="name x y body_mesh body_z wheel_mesh wheel_x wheel_y">
     <!-- The mount frame is at the rolling-wheel center and swivels about z. -->
     <link name="${name}_mount">
-      <visual name="cad_body_visual">
+      <visual>
         <origin xyz="0 0 ${body_z}" rpy="0 0 0"/>
         <geometry><mesh filename="package://amr_description/meshes/${body_mesh}"/></geometry>
@@ -102,6 +122,7 @@
       <dynamics damping="0.05" friction="0.01"/>
     </joint>
+    <xacro:exclude_lidar_self_visuals link="${name}_mount"/>
     <link name="${name}_wheel">
-      <visual name="cad_wheel_visual">
+      <visual>
         <origin xyz="0 0 0" rpy="-1.57079632679 0 0"/>
         <geometry><mesh filename="package://amr_description/meshes/${wheel_mesh}"/></geometry>
@@ -124,9 +145,10 @@
       <mu2>0.01</mu2>
     </gazebo>
+    <xacro:exclude_lidar_self_visuals link="${name}_wheel"/>
   </xacro:macro>
   <link name="base_footprint"/>
   <link name="base_link">
     <!-- Derived CAD visual; the primitive collision preserves the footprint, bottom -0.02, and top 0.33. -->
-    <visual name="cad_visual">
+    <visual>
       <origin xyz="0 0 0" rpy="0 0 0"/>
       <geometry><mesh filename="package://amr_description/meshes/base_link.STL"/></geometry>
@@ -145,4 +167,5 @@
     <origin xyz="0 0 ${base_footprint_height}"/>
   </joint>
+  <xacro:exclude_lidar_self_visuals link="base_link"/>
   <!-- Generic payload remains base-only default-on at its existing support height. -->
   <xacro:if value="$(arg include_generic_payload)">
@@ -162,4 +185,5 @@
       <origin xyz="0 0 ${generic_payload_support_top_z + generic_payload_clearance + payload_z_checked / 2.0}"/>
     </joint>
+    <xacro:exclude_lidar_self_visuals link="payload_link"/>
   </xacro:if>
   <xacro:drive_wheel name="left_wheel" y="${wheel_separation / 2.0}" rpy="-1.57079632679" axis_z="1"/>
@@ -195,7 +219,8 @@
     <origin xyz="0 0 0.18"/>
   </joint>
+  <xacro:exclude_lidar_self_visuals link="imu_link"/>
   <!-- CAD LiDAR poses are retained as the software frame contract. -->
   <link name="front_lidar_link">
-    <visual name="cad_visual">
+    <visual>
       <origin xyz="0 0 0" rpy="0 0 0"/>
       <geometry><mesh filename="package://amr_description/meshes/lidar_front_link.STL"/></geometry>
@@ -211,5 +236,5 @@
   </joint>
   <link name="rear_lidar_link">
-    <visual name="cad_visual">
+    <visual>
       <origin xyz="0 0 0" rpy="0 0 0"/>
       <geometry><mesh filename="package://amr_description/meshes/lidar_back_link.STL"/></geometry>
@@ -235,4 +260,5 @@
         </scan>
         <range><min>0.2</min><max>20.0</max><resolution>0.01</resolution></range>
+        <visibility_mask>${lidar_visibility_mask}</visibility_mask>
       </lidar>
     </sensor>
@@ -249,7 +275,10 @@
         </scan>
         <range><min>0.2</min><max>20.0</max><resolution>0.01</resolution></range>
+        <visibility_mask>${lidar_visibility_mask}</visibility_mask>
       </lidar>
     </sensor>
   </gazebo>
+  <xacro:exclude_lidar_self_visuals link="front_lidar_link"/>
+  <xacro:exclude_lidar_self_visuals link="rear_lidar_link"/>
   <gazebo reference="imu_link">
     <sensor name="imu" type="imu">

File: src/amr_description/urdf/phase14_mobile_manipulator.urdf.xacro (robot description, xacro)
@@ -23,4 +23,11 @@
     <origin xyz="0 0 0.33" rpy="0 0 0"/>
   </joint>
+  <xacro:exclude_lidar_self_visuals link="arm_base_link"/>
+  <xacro:exclude_lidar_self_visuals link="arm_link_1"/>
+  <xacro:exclude_lidar_self_visuals link="arm_link_2"/>
+  <xacro:exclude_lidar_self_visuals link="arm_link_3"/>
+  <xacro:exclude_lidar_self_visuals link="arm_link_4"/>
+  <xacro:exclude_lidar_self_visuals link="arm_link_5"/>
+  <xacro:exclude_lidar_self_visuals link="arm_link_6"/>
   <link name="gripper_base_link">
     <visual><geometry><box size="0.10 0.10 0.04"/></geometry></visual>
@@ -53,4 +60,7 @@
     <mimic joint="gripper_finger_joint" multiplier="1.0" offset="0.0"/>
   </joint>
+  <xacro:exclude_lidar_self_visuals link="gripper_base_link"/>
+  <xacro:exclude_lidar_self_visuals link="gripper_left_finger_link"/>
+  <xacro:exclude_lidar_self_visuals link="gripper_right_finger_link"/>
   <link name="gripper_tcp"/>
   <joint name="gripper_tcp_joint" type="fixed">
@@ -113,4 +123,5 @@
     <origin xyz="0.25 0.20 0.65" rpy="0 0 0"/>
   </joint>
+  <xacro:exclude_lidar_self_visuals link="product_camera_link"/>
   <link name="product_camera_optical_frame"/>
   <joint name="product_camera_optical_joint" type="fixed">
@@ -141,4 +152,5 @@
       <origin xyz="0.15 0 0"/>
     </joint>
+    <xacro:exclude_lidar_self_visuals link="stowed_product_link"/>
   </xacro:if>
   <ros2_control name="Phase14MobileManipulatorSystem" type="system">
